Commit message: make xacro gazebo ready

File: moveit_ws/src/so101_moveit_config/config/so101.ros2_control.xacro (robot description, xacro)
@@ -1,10 +1,10 @@
 <?xml version="1.0"?>
 <robot xmlns:xacro="http://www.ros.org/wiki/xacro">
-    <xacro:macro name="so101_ros2_control" params="name initial_positions_file">
+    <xacro:macro name="so101_ros2_control" params="name initial_positions_file hardware_plugin:='mock_components/GenericSystem'">
         <xacro:property name="initial_positions" value="${xacro.load_yaml(initial_positions_file)['initial_positions']}"/>
         <ros2_control name="${name}" type="system">
             <hardware>
-                <!-- By default, set up controllers for simulation. This won't work on real hardware -->
-                <plugin>mock_components/GenericSystem</plugin>
+                <!-- Mock by default; sim passes the Gazebo system instead. -->
+                <plugin>${hardware_plugin}</plugin>
             </hardware>
             <joint name="shoulder_pan">

File: moveit_ws/src/so101_moveit_config/config/so101.urdf.xacro (robot description, xacro)
@@ -2,8 +2,36 @@
 <robot xmlns:xacro="http://www.ros.org/wiki/xacro" name="so101">
     <xacro:arg name="initial_positions_file" default="initial_positions.yaml" />
+    <!-- sim:=true swaps the ros2_control hardware for Gazebo's and adds the
+         simulation-only tags below. Default keeps mock hardware, so every
+         existing MoveIt launch file behaves exactly as before. -->
+    <xacro:arg name="sim" default="false" />
     <!-- Import so101 urdf file -->
     <xacro:include filename="$(find so101_description)/urdf/so101.urdf" />
     <!-- Import control_xacro -->
     <xacro:include filename="so101.ros2_control.xacro" />
-    <xacro:so101_ros2_control name="FakeSystem" initial_positions_file="$(arg initial_positions_file)"/>
+    <xacro:property name="sim" value="$(arg sim)" />
+    <xacro:property name="hardware_plugin"
+        value="${'gz_ros2_control/GazeboSimSystem' if sim else 'mock_components/GenericSystem'}" />
+    <xacro:so101_ros2_control name="So101System"
+        initial_positions_file="$(arg initial_positions_file)"
+        hardware_plugin="${hardware_plugin}" />
+    <xacro:if value="$(arg sim)">
+        <!-- Gazebo needs a real fixed joint to a static link. The SRDF
+             virtual_joint tells MoveIt where the base is but anchors nothing,
+             so without this the arm is a free body and falls on tick one. -->
+        <link name="world" />
+        <joint name="world_joint" type="fixed">
+            <parent link="world" />
+            <child link="base_link" />
+            <origin xyz="0 0 0" rpy="0 0 0" />
+        </joint>
+        <!-- Runs controller_manager inside the Gazebo process, so its update
+             loop is driven by simulation time rather than wall clock. -->
+        <gazebo>
+            <plugin filename="libgz_ros2_control-system.so"
+                    name="gz_ros2_control::GazeboSimROS2ControlPlugin">
+                <parameters>$(find so101_moveit_config)/config/ros2_controllers.yaml</parameters>
+            </plugin>
+        </gazebo>
+    </xacro:if>
 </robot>

Commit message: add so101_hardware SystemInterface for the Feetech STS3215 bus

File: moveit_ws/src/so101_moveit_config/config/so101.ros2_control.xacro (robot description, xacro)
@@ -1,10 +1,16 @@
 <?xml version="1.0"?>
 <robot xmlns:xacro="http://www.ros.org/wiki/xacro">
-    <xacro:macro name="so101_ros2_control" params="name initial_positions_file hardware_plugin:='mock_components/GenericSystem'">
+    <xacro:macro name="so101_ros2_control" params="name initial_positions_file hardware_plugin:='mock_components/GenericSystem' device:='/dev/ttyACM0' baud:='1000000' calib_file:='so101_follower_calib.json' torque_limit:='300' enable_torque:='true'">
         <xacro:property name="initial_positions" value="${xacro.load_yaml(initial_positions_file)['initial_positions']}"/>
         <ros2_control name="${name}" type="system">
             <hardware>
-                <!-- Mock by default; sim passes the Gazebo system instead. -->
                 <plugin>${hardware_plugin}</plugin>
+                <xacro:if value="${hardware_plugin == 'so101_hardware/So101System'}">
+                    <param name="device">${device}</param>
+                    <param name="baud">${baud}</param>
+                    <param name="calib_file">${calib_file}</param>
+                    <param name="torque_limit">${torque_limit}</param>
+                    <param name="enable_torque">${enable_torque}</param>
+                </xacro:if>
             </hardware>
             <joint name="shoulder_pan">

File: moveit_ws/src/so101_moveit_config/config/so101.urdf.xacro (robot description, xacro)
@@ -2,22 +2,26 @@
 <robot xmlns:xacro="http://www.ros.org/wiki/xacro" name="so101">
     <xacro:arg name="initial_positions_file" default="initial_positions.yaml" />
-    <!-- sim:=true swaps the ros2_control hardware for Gazebo's and adds the
-         simulation-only tags below. Default keeps mock hardware, so every
-         existing MoveIt launch file behaves exactly as before. -->
-    <xacro:arg name="sim" default="false" />
+    <xacro:arg name="hardware" default="mock" />
+    <xacro:arg name="device" default="/dev/ttyACM0" />
+    <xacro:arg name="baud" default="1000000" />
+    <xacro:arg name="calib_file" default="so101_follower_calib.json" />
+    <xacro:arg name="torque_limit" default="300" />
+    <xacro:arg name="enable_torque" default="true" />
     <!-- Import so101 urdf file -->
     <xacro:include filename="$(find so101_description)/urdf/so101.urdf" />
     <!-- Import control_xacro -->
     <xacro:include filename="so101.ros2_control.xacro" />
-    <xacro:property name="sim" value="$(arg sim)" />
-    <!-- `sim` here is the property from above, which xacro has already coerced
-         to a bool. Comparing it against the string 'true' silently fails.
-         We need to use the property name, not the string value. -->
+    <xacro:property name="hardware" value="$(arg hardware)" />
     <xacro:property name="hardware_plugin"
-        value="${'gz_ros2_control/GazeboSimSystem' if sim else 'mock_components/GenericSystem'}" />
+        value="${'gz_ros2_control/GazeboSimSystem' if hardware == 'gazebo' else ('so101_hardware/So101System' if hardware == 'real' else 'mock_components/GenericSystem')}" />
     <xacro:so101_ros2_control name="So101System"
         initial_positions_file="$(arg initial_positions_file)"
-        hardware_plugin="${hardware_plugin}" />
-    <xacro:if value="$(arg sim)">
+        hardware_plugin="${hardware_plugin}"
+        device="$(arg device)"
+        baud="$(arg baud)"
+        calib_file="$(arg calib_file)"
+        torque_limit="$(arg torque_limit)"
+        enable_torque="$(arg enable_torque)" />
+    <xacro:if value="${hardware == 'gazebo'}">
         <!-- Gazebo needs a real fixed joint to a static link. The SRDF
              virtual_joint tells MoveIt where the base is but anchors nothing,
